Commit message: urdf: basic robot layout

File: urdf/mbot_ranger_dashing_raptor.urdf.xacro (robot description, xacro)
@@ -10,6 +10,4 @@
   <xacro:include filename="$(find mbot_description)/urdf/mbot_ranger_dashing_raptor/mbot_ranger_dashing_raptor_macro.xacro"/>
   <xacro:include filename="$(find mbot_description)/urdf/mbot_ranger_dashing_raptor/mbot_ranger_dashing_raptor_macro.ros2_control.xacro"/>
-  <!-- create link fixed to the "world" -->
-  <link name="world" />
   <!-- Load robot's macro with parameters -->
   <!-- set prefix if multiple robots are used -->

File: urdf/mbot_ranger_dashing_raptor/mbot_ranger_dashing_raptor_macro.ros2_control.xacro (robot description, xacro)
@@ -38,48 +38,4 @@
       </joint>
       <joint name="${prefix}joint2">
-        <command_interface name="position">     <!-- Add/Remove interfaces as needed -->
-          <param name="min">-1</param>
-          <param name="max">1</param>
-        </command_interface>
-        <state_interface name="position">
-          <param name="initial_value">0.0</param>
-        </state_interface>
-        <state_interface name="velocity"/>
-        <state_interface name="acceleration"/>
-      </joint>
-      <joint name="${prefix}joint3">
-        <command_interface name="position">     <!-- Add/Remove interfaces as needed -->
-          <param name="min">-1</param>
-          <param name="max">1</param>
-        </command_interface>
-        <state_interface name="position">
-          <param name="initial_value">0.0</param>
-        </state_interface>
-        <state_interface name="velocity"/>
-        <state_interface name="acceleration"/>
-      </joint>
-      <joint name="${prefix}joint4">
-        <command_interface name="position">     <!-- Add/Remove interfaces as needed -->
-          <param name="min">-1</param>
-          <param name="max">1</param>
-        </command_interface>
-        <state_interface name="position">
-          <param name="initial_value">0.0</param>
-        </state_interface>
-        <state_interface name="velocity"/>
-        <state_interface name="acceleration"/>
-      </joint>
-      <joint name="${prefix}joint5">
-        <command_interface name="position">     <!-- Add/Remove interfaces as needed -->
-          <param name="min">-1</param>
-          <param name="max">1</param>
-        </command_interface>
-        <state_interface name="position">
-          <param name="initial_value">0.0</param>
-        </state_interface>
-        <state_interface name="velocity"/>
-        <state_interface name="acceleration"/>
-      </joint>
-      <joint name="${prefix}joint6">
         <command_interface name="position">     <!-- Add/Remove interfaces as needed -->
           <param name="min">-1</param>

File: urdf/mbot_ranger_dashing_raptor/mbot_ranger_dashing_raptor_macro.xacro (robot description, xacro)
@@ -12,5 +12,5 @@
         <origin xyz="0 0 0" rpy="0 0 0" />
         <geometry>
-          <cylinder length="0.3" radius="0.3" />
+          <box size="0.025 0.125 0.025" />
 <!--           <mesh filename="package://mbot_description/meshes/mbot_ranger_dashing_raptor/visual/base_link.dae" /> -->
         </geometry>
@@ -19,11 +19,30 @@
         <origin xyz="0 0 0" rpy="0 0 0" />
         <geometry>
-          <cylinder length="0.3" radius="0.3" />
+          <box size="0.025 0.125 0.025" />
 <!--           <mesh filename="package://mbot_description/meshes/mbot_ranger_dashing_raptor/collision/base_link.stl" /> -->
         </geometry>
       </collision>
     </link>
-    <!-- link 1 -->
-    <link name="${prefix}link1">
+    <link name="${prefix}chassis">
+      <!-- Default inertial for Gazebo/Ingnition - copy and edit block from 'common.xacro'
+           to get more realistic behaviour-->
+      <xacro:default_inertial/>
+      <visual>
+        <origin xyz="0.07 0 0" rpy="0 0 0" />
+        <geometry>
+          <box size="0.14 0.125 0.025" />
+<!--           <mesh filename="package://mbot_description/meshes/mbot_ranger_dashing_raptor/visual/base_link.dae" /> -->
+        </geometry>
+      </visual>
+      <collision>
+        <origin xyz="0.07 0 0" rpy="0 0 0" />
+        <geometry>
+          <box size="0.14 0.125 0.025" />
+<!--           <mesh filename="package://mbot_description/meshes/mbot_ranger_dashing_raptor/collision/base_link.stl" /> -->
+        </geometry>
+      </collision>
+    </link>
+    <!-- left  wheel -->
+    <link name="${prefix}caster_wheel">
       <!-- Default inertial for Gazebo/Ingnition - copy and edit block from 'common.xacro'
            to get more realistic behaviour-->
@@ -32,6 +51,6 @@
         <origin xyz="0 0 0" rpy="0 0 0" />
         <geometry>
-          <cylinder length="0.3" radius="0.15" />
-<!--           <mesh filename="package://mbot_description/meshes/mbot_ranger_dashing_raptor/visual/link1.dae" /> -->
+          <sphere radius="0.01" />
+<!--           <mesh filename="package://mbot_description/meshes/mbot_ranger_dashing_raptor/visual/left_wheel.dae" /> -->
         </geometry>
       </visual>
@@ -39,197 +58,80 @@
         <origin xyz="0 0 0" rpy="0 0 0" />
         <geometry>
-          <cylinder length="0.3" radius="0.15" />
-<!--           <mesh filename="package://mbot_description/meshes/mbot_ranger_dashing_raptor/collision/link1.stl" /> -->
+          <sphere radius="0.01" />
+<!--           <mesh filename="package://mbot_description/meshes/mbot_ranger_dashing_raptor/collision/left_wheel.stl" /> -->
         </geometry>
       </collision>
     </link>
-    <!-- link 2 -->
-    <link name="${prefix}link2">
+    <!-- left  wheel -->
+    <link name="${prefix}left_wheel">
       <!-- Default inertial for Gazebo/Ingnition - copy and edit block from 'common.xacro'
            to get more realistic behaviour-->
       <xacro:default_inertial/>
       <visual>
-        <origin xyz="0 0 0" rpy="0 0 0" />
+        <origin xyz="0 0.008 0" rpy="0 ${pi/2} ${pi/2}" />
         <geometry>
-          <cylinder length="0.8" radius="0.15" />
-<!--           <mesh filename="package://mbot_description/meshes/mbot_ranger_dashing_raptor/visual/link2.dae" /> -->
+          <cylinder length="0.016" radius="0.0325" />
+<!--           <mesh filename="package://mbot_description/meshes/mbot_ranger_dashing_raptor/visual/left_wheel.dae" /> -->
         </geometry>
       </visual>
       <collision>
-        <origin xyz="0 0 0" rpy="0 0 0" />
+        <origin xyz="0 0.008 0" rpy="0 ${pi/2} ${pi/2}" />
         <geometry>
-          <cylinder length="0.8" radius="0.15" />
-<!--           <mesh filename="package://mbot_description/meshes/mbot_ranger_dashing_raptor/collision/link2.stl"  /> -->
+          <cylinder length="0.016" radius="0.0325" />
+<!--           <mesh filename="package://mbot_description/meshes/mbot_ranger_dashing_raptor/collision/left_wheel.stl" /> -->
         </geometry>
       </collision>
     </link>
-    <!-- link 3 -->
-    <link name="${prefix}link3">
+    <!-- right wheel -->
+    <link name="${prefix}right_wheel">
       <!-- Default inertial for Gazebo/Ingnition - copy and edit block from 'common.xacro'
            to get more realistic behaviour-->
       <xacro:default_inertial/>
       <visual>
-        <origin xyz="0 0 0" rpy="0 0 0" />
+        <origin xyz="0 -0.008 0" rpy="0 ${pi/2} ${pi/2}" />
         <geometry>
-          <cylinder length="0.5" radius="0.10" />
-<!--           <mesh filename="package://mbot_description/meshes/mbot_ranger_dashing_raptor/visual/link3.dae" /> -->
+          <cylinder length="0.016" radius="0.0325" />
+<!--           <mesh filename="package://mbot_description/meshes/mbot_ranger_dashing_raptor/visual/right_wheel.dae" /> -->
         </geometry>
       </visual>
       <collision>
-        <origin xyz="0 0 0" rpy="0 0 0" />
+        <origin xyz="0 -0.008 0" rpy="0 ${pi/2} ${pi/2}" />
         <geometry>
-          <cylinder length="0.5" radius="0.10" />
-<!--           <mesh filename="package://mbot_description/meshes/mbot_ranger_dashing_raptor/collision/link3.stl"  /> -->
+          <cylinder length="0.016" radius="0.0325" />
+<!--           <mesh filename="package://mbot_description/meshes/mbot_ranger_dashing_raptor/collision/right_wheel.stl"  /> -->
         </geometry>
       </collision>
     </link>
-    <!-- link 4 -->
-    <link name="${prefix}link4">
-      <!-- Default inertial for Gazebo/Ingnition - copy and edit block from 'common.xacro'
-           to get more realistic behaviour-->
-      <xacro:default_inertial/>
-      <visual>
-        <origin xyz="0 0 0" rpy="0 0 0" />
-        <geometry>
-          <cylinder length="0.1" radius="0.2" />
-<!--           <mesh filename="package://mbot_description/meshes/mbot_ranger_dashing_raptor/visual/link4.dae" /> -->
-        </geometry>
-      </visual>
-      <collision>
-        <origin xyz="0 0 0" rpy="0 0 0" />
-        <geometry>
-          <cylinder length="0.1" radius="0.2" />
-<!--           <mesh filename="package://mbot_description/meshes/mbot_ranger_dashing_raptor/collision/link4.stl"  /> -->
-        </geometry>
-      </collision>
-    </link>
-    <!-- link 5 -->
-    <link name="${prefix}link5">
-      <!-- Default inertial for Gazebo/Ingnition - copy and edit block from 'common.xacro'
-           to get more realistic behaviour-->
-      <xacro:default_inertial/>
-      <visual>
-        <origin xyz="0 0 0" rpy="0 0 0" />
-        <geometry>
-          <cylinder length="0.2" radius="0.1" />
-<!--           <mesh filename="package://mbot_description/meshes/mbot_ranger_dashing_raptor/visual/link5.dae" /> -->
-        </geometry>
-      </visual>
-      <collision>
-        <origin xyz="0 0 0" rpy="0 0 0" />
-        <geometry>
-          <cylinder length="0.2" radius="0.1" />
-<!--           <mesh filename="package://mbot_description/meshes/mbot_ranger_dashing_raptor/collision/link5.stl" /> -->
-        </geometry>
-      </collision>
-    </link>
-    <!-- link 6 -->
-    <link name="${prefix}link6">
-      <!-- Default inertial for Gazebo/Ingnition - copy and edit block from 'common.xacro'
-           to get more realistic behaviour-->
-      <xacro:default_inertial/>
-      <visual>
-        <origin xyz="0 0 0" rpy="0 0 0" />
-        <geometry>
-          <cylinder length="0.05" radius="0.1" />
-<!--           <mesh filename="package://mbot_description/meshes/mbot_ranger_dashing_raptor/visual/link6.dae" /> -->
-        </geometry>
-      </visual>
-      <collision>
-        <origin xyz="0 0 0" rpy="0 0 0" />
-        <geometry>
-          <cylinder length="0.05" radius="0.1" />
-<!--           <mesh filename="package://mbot_description/meshes/mbot_ranger_dashing_raptor/collision/link6.stl" /> -->
-        </geometry>
-      </collision>
-    </link>
-    <!-- All-zero tool frame. This frame should correspond to the TOOL frame of the robot's controller.) -->
-    <link name="${prefix}tool0" />
-    <!-- tool link -->
-<!-- START Delete if not needed -->
-    <!-- Standard frames for industrial robots. Also useful for manipulators.
-         (ROS-I specs - https://wiki.ros.org/Industrial/Tutorials/WorkingWithRosIndustrialRobotSupportPackages#Standardised_links_.2F_frames)-->
-    <!-- This frame should correspond to the BASE coordinate system of robot's controller.) -->
-    <link name="${prefix}base" />
-    <!-- Frame for mounting EEF models to a manipulator. x+ axis points forward (REP 103). -->
-    <link name="${prefix}flange" />
-<!-- END Delete if not needed  -->
     <!-- END LINKS -->
     <!-- JOINTS -->
-    <!-- base_joint fixes base_link to the environment -->
-    <joint name="${prefix}base_joint" type="fixed">
-      <xacro:insert_block name="origin" />
-      <parent link="${parent}" />
-      <child link="${prefix}base_link" />
+    <joint name="${prefix}fixture1" type="fixed">
+      <origin xyz="0.025 0 0.04" rpy="0 0 0" />
+      <parent link="${prefix}base_link" />
+      <child link="${prefix}chassis" />
+      <axis xyz="0 0 1" />
+    </joint>
+    <joint name="${prefix}fixture2" type="fixed">
+      <origin xyz="0.14 0 -0.0625" rpy="0 0 0" /> <!-- should touch ground while chassis is level -->
+      <parent link="${prefix}chassis" />
+      <child link="${prefix}caster_wheel" />
+      <axis xyz="0 0 1" />
     </joint>
     <!-- joint 1 -->
     <joint name="${prefix}joint1" type="revolute">
-      <origin xyz="0 0 0.3" rpy="${pi} 0 0" />
+      <origin xyz="0 -0.0625 0" rpy="0 0 0" />
       <parent link="${prefix}base_link" />
-      <child link="${prefix}link1" />
-      <axis xyz="0 0 1" />
+      <child link="${prefix}right_wheel" />
+      <axis xyz="0 1 0" />
       <limit effort="0" lower="${radians(-180)}" upper="${radians(180)}" velocity="${radians(180)}" />
     </joint>
     <!-- joint 2 -->
     <joint name="${prefix}joint2" type="revolute">
-      <origin xyz="0 0 0.3" rpy="${pi/2} 0 0" />
-      <parent link="${prefix}link1" />
-      <child link="${prefix}link2" />
-      <axis xyz="0 0 1" />
+      <origin xyz="0 0.0625 0" rpy="0 0 0" />
+      <parent link="${prefix}base_link" />
+      <child link="${prefix}left_wheel" />
+      <axis xyz="0 1 0" />
       <limit effort="0" lower="${radians(-180)}" upper="${radians(180)}" velocity="${radians(180)}" />
     </joint>
-    <!-- joint 3 -->
-    <joint name="${prefix}joint3" type="revolute">
-      <origin xyz="0.8 0 0" rpy="0 0 0" />
-      <parent link="${prefix}link2" />
-      <child link="${prefix}link3" />
-      <axis xyz="0 0 1" />
-      <limit effort="0" lower="${radians(-90)}" upper="${radians(180)}" velocity="${radians(270)}" />
-    </joint>
-    <!-- joint 4 -->
-    <joint name="${prefix}joint4" type="revolute">
-      <origin xyz="0 0.1 0" rpy="0 ${-pi/2} 0" />
-      <parent link="${prefix}link3" />
-      <child link="${prefix}link4" />
-      <axis xyz="0 0 1" />
-      <limit effort="0" lower="${radians(-360)}" upper="${radians(360)}" velocity="${radians(360)}" />
-    </joint>
-    <!-- joint 5 -->
-    <joint name="${prefix}joint5" type="revolute">
-      <origin xyz="0 0 -0.1" rpy="0 ${pi/2} 0" />
-      <parent link="${prefix}link4" />
-      <child link="${prefix}link5" />
-      <axis xyz="0 0 1" />
-      <limit effort="0" lower="${radians(-120)}" upper="${radians(120)}" velocity="${radians(540)}" />
-    </joint>
-    <!-- joint 6 -->
-    <joint name="${prefix}joint6" type="revolute">
-      <origin xyz="0 0 0.1" rpy="0 ${-pi/2} 0" />
-      <parent link="${prefix}link5" />
-      <child link="${prefix}link6" />
-      <axis xyz="0 0 1" />
-      <limit effort="0" lower="${radians(-360)}" upper="${radians(360)}" velocity="${radians(720)}" />
-    </joint>
-    <!-- tool frame - fixed frame -->
-    <joint name="${prefix}joint6-tool0" type="fixed">
-      <parent link="${prefix}link6" />
-      <child link="${prefix}tool0" />
-      <origin xyz="0 0 -0.115" rpy="0 ${-pi} ${-pi/2}" />
-    </joint>
     <!-- END JOINTS -->
-<!-- START Delete if not needed -->
-    <!-- Standard frames for industrial robots. Also useful for manipulators.
-         (ROS-I specs - https://wiki.ros.org/Industrial/Tutorials/WorkingWithRosIndustrialRobotSupportPackages#Standardised_links_.2F_frames)-->
-    <joint name="${prefix}base_link-base_joint" type="fixed">
-      <origin xyz="0 0 0" rpy="0 0 0" />
-      <parent link="${prefix}base_link" />
-      <child link="${prefix}base" />
-    </joint>
-    <joint name="${prefix}tool0-flange_joint" type="fixed">
-      <origin xyz="0 0 0" rpy="0 0 0" />
-      <parent link="${prefix}tool0" />
-      <child link="${prefix}flange" />
-    </joint>
-<!-- END Delete if not needed  -->
   </xacro:macro>
 </robot>

Commit message: urdf: add some color

File: urdf/mbot_ranger_dashing_raptor.urdf.xacro (robot description, xacro)
@@ -8,4 +8,16 @@
   <xacro:arg name="sim_gazebo" default="false" />
   <xacro:arg name="simulation_controllers" default="" />
+  <material name="white">
+    <color rgba="1 1 1 1"/>
+  </material>
+  <material name="orange">
+    <color rgba="1 0.3 0.1 1"/>
+  </material>
+  <material name="blue">
+    <color rgba="0.2 0.2 1 1"/>
+  </material>
+  <material name="black">
+    <color rgba="0 0 0 1"/>
+  </material>
   <xacro:include filename="$(find mbot_description)/urdf/mbot_ranger_dashing_raptor/mbot_ranger_dashing_raptor_macro.xacro"/>
   <xacro:include filename="$(find mbot_description)/urdf/mbot_ranger_dashing_raptor/mbot_ranger_dashing_raptor_macro.ros2_control.xacro"/>

File: urdf/mbot_ranger_dashing_raptor/mbot_ranger_dashing_raptor_macro.xacro (robot description, xacro)
@@ -15,4 +15,5 @@
 <!--           <mesh filename="package://mbot_description/meshes/mbot_ranger_dashing_raptor/visual/base_link.dae" /> -->
         </geometry>
+        <material name="blue" />
       </visual>
       <collision>
@@ -34,4 +35,5 @@
 <!--           <mesh filename="package://mbot_description/meshes/mbot_ranger_dashing_raptor/visual/base_link.dae" /> -->
         </geometry>
+        <material name="blue" />
       </visual>
       <collision>
@@ -43,5 +45,5 @@
       </collision>
     </link>
-    <!-- left  wheel -->
+    <!-- caster  wheel -->
     <link name="${prefix}caster_wheel">
       <!-- Default inertial for Gazebo/Ingnition - copy and edit block from 'common.xacro'
@@ -54,4 +56,5 @@
 <!--           <mesh filename="package://mbot_description/meshes/mbot_ranger_dashing_raptor/visual/left_wheel.dae" /> -->
         </geometry>
+        <material name="black" />
       </visual>
       <collision>
@@ -74,4 +77,5 @@
 <!--           <mesh filename="package://mbot_description/meshes/mbot_ranger_dashing_raptor/visual/left_wheel.dae" /> -->
         </geometry>
+        <material name="black" />
       </visual>
       <collision>
@@ -94,4 +98,5 @@
 <!--           <mesh filename="package://mbot_description/meshes/mbot_ranger_dashing_raptor/visual/right_wheel.dae" /> -->
         </geometry>
+        <material name="black" />
       </visual>
       <collision>
